Commit message: Benchmark control

File: hardware/benchmark/robot.urdf (robot description, URDF)
Before this commit: robot benchmark, 10 links, 9 joints
Links:
- removed link left_tibia
- added link inner_knee, mass 0.139137; visual mesh filename=package://assets/ankle_bearing_cover.stl; visual mesh filename=package://assets/ankle_bearing_cover.stl
- link aluminum_profile: geometry visual mesh filename=package://assets/aluminum_profile.stl; visual mesh filename=package://assets/bearing_6804_2rs.stl
- link ankle_shaft: geometry visual mesh filename=package://assets/ankle_shaft.stl; visual mesh filename=package://assets/p210fm_plain_bearing.stl
- link benchmark_foot: geometry visual mesh filename=package://assets/ankle_alu.stl; visual mesh filename=package://assets/ankle_alu.stl
- link left_crank: geometry visual mesh filename=package://assets/bearing_6804_2rs.stl; visual mesh filename=package://assets/din_6325_3mm__configuration__6.stl
- link motor_pulley: geometry visual mesh filename=package://assets/din_6325_3mm__configuration__12.stl; visual mesh filename=package://assets/motor_pulley.stl
- link motor_pulley_2: geometry visual mesh filename=package://assets/din_6325_3mm__configuration__12.stl; visual mesh filename=package://assets/motor_pulley.stl
Joints:
- joint ankle_joint: origin xyz=-3.31207e-14 -0.15 -0.0503 rpy=3.14159 8.42708e-16 3.14159 -> xyz=5.42101e-20 -0.15 -0.0503 rpy=3.14159 2.1445e-17 -3.14159; parent left_tibia -> inner_knee
- joint ankle_passive: origin xyz=-1.42561e-14 -1.11022e-15 -0.005 rpy=1.98711e-16 -7.13893e-17 -1.5708 -> xyz=0 0 -0.005 rpy=1.65388e-31 -2.80452e-29 -1.5708; parent left_tibia -> inner_knee
- joint closing_crank_frame: origin xyz=-0.15 0.05 -0.0068 rpy=1.5708 -6.1175e-15 -1.7919e-15 -> xyz=-0.15 0.05 -0.0068 rpy=1.5708 -6.11275e-15 -1.50324e-15
- joint closing_foot_frame: origin xyz=0.025 -1.94289e-16 -0.0232 rpy=1.5708 -2.0777e-16 -3.14159 -> xyz=0.025 -1.11022e-16 -0.0232 rpy=1.5708 -1.80862e-16 -3.14159
- joint foot_frame: origin xyz=-0.00573895 -0.0515 -0.0197 rpy=1.5708 7.63818e-30 -3.14159 -> xyz=-0.00573895 -0.0515 -0.0197 rpy=1.5708 -1.89761e-17 -3.14159
- joint knee_joint: child left_tibia -> inner_knee; origin xyz=-0.000132957 -0.0835 0.269 rpy=1.5708 3.18659e-18 2.27523e-16 -> xyz=-0.000132957 -0.0835 0.269 rpy=1.5708 -0 1.64748e-23
- joint upper_crank: origin xyz=-5.76761e-14 0.025 -0.029 rpy=-3.14159 -9.93684e-16 2.49809 -> xyz=-4.14113e-14 0.025 -0.029 rpy=3.14159 -1.67015e-15 2.49809
